Commit message: feat: add left hand asset, modify bvh_rerun_vis for bimanual visualization

File: assets/rh56dftp/rh56dftp_modified_right.urdf (robot description, URDF)
Before this commit: robot Rhand, 32 links, 31 joints
Links:
- removed link human_wrist_link
- added link right_wrist_link; visual sphere radius=0.001
Joints:
- removed joint human_wrist_joint
- added joint right_wrist_joint: type fixed, parent right_base_link, child right_wrist_link, origin xyz=-0.015 0.0 0.05 rpy=0 0 0
